File: pcb-project-s.kicad_sch (KiCad schematic)
At the start: 29 parts, among them SW1 SW_Push, U1 ATmega32U4-A, U2 PRTR5V0U2X, Y1 16MHz

Commit message: Designed the PCB
Parts:
- removed MX1, MX2, MX3, MX4: MX-NoLED, MX_Alps_Hybrid:MX-1U-NoLED, symbol MX_Alps_Hybrid:MX-NoLED
- removed R2, R3: 22, Resistor_SMD:R_0805_2012Metric, symbol Device:R_Small
- added MX1, MX2, MX3, MX4: MX-LED, MX_Alps_Hybrid:MX-1U, symbol MX_Alps_Hybrid:MX-LED
Connections:
- net D+ is gone; now on an unnamed net: R6.2
- net D- is gone; now on an unnamed net: R5.2
- net COL0: now also MX1.1 (COL), MX2.1 (COL)
- net COL1: now also MX3.1 (COL), MX4.1 (COL)
- net GND: now also R8.1
- net at D3.2 (A): now also MX2.2 (ROW)
- net at D1.2 (A): now also MX1.2 (ROW)
- net at D2.2 (A): now also MX3.2 (ROW)
- net at D4.2 (A): now also MX4.2 (ROW)
